File: Breadboard_14_Rows_Power_Supply_V1.kicad_pcb (KiCad board)
At the start: 2 copper layers, 29.2 x 51.8 mm, 18 parts, among them J1 Barrel_Jack_Switch, J2 Conn_02x02_Odd_Even, J3 Conn_02x02_Odd_Even, SW1 SW_DPDT_x2, U1 LM7805_TO220

Commit message: Routing with Freerouting.jar, rest ist the same as in the master branch
Parts:
- renumbered REF** to REF_Kicad
Routing:
- net GND: track 90.4 -> 0.00 mm
- net /Vout1: track 38.0 -> 34.8 mm
- net /Vout2: track 58.6 -> 56.8 mm
- net /Vin: track 35.5 -> 34.0 mm
- net /V2: track 36.5 -> 35.4 mm
